File: heartthingv2.kicad_sch (KiCad schematic)
At the start: 38 parts, among them J1 Conn_01x03_Socket, J2 Conn_01x09_Pin, J3 Conn_01x02_Socket, U1 MAX30003CTI_, U2 AP2112K-1.8, U3 TXB0108PW, U4 102010469, U5 MAX17048G_T10, Y1 Crystal_GND23

Commit message: no diddy
Parts:
- removed C11: 10 uF, symbol Device:C
- added C22: 3.9 pF, symbol Device:C
- added C23, C24, C25, C26: 100 nF, symbol Device:C
- added C27, C36: 10 uF, symbol Device:C
- added C28, C29: 2.2 uF, symbol Device:C
- added C30: 10 nF, symbol Device:C
- added C31: 2.2 nF, symbol Device:C
- added C32: 1.5 pF, symbol Device:C
- added C33: 2.0 pF, symbol Device:C
- added C34: 0.3 pF, symbol Device:C
- added C35: C, symbol Device:C
- added D1: D, symbol Device:D
- added FB1: 120, symbol Device:FerriteBead
- added J4: USB_C_Receptacle_USB2.0_16P, symbol Connector:USB_C_Receptacle_USB2.0_16P
- added L1: 4.7 uH, symbol Device:L
- added L2: 2.7 nH, symbol Device:L
- added L3, L4: 3.5 nH, symbol Device:L
- added R7: 1k, 0201, symbol Device:R
- added U6: NRF54L15-QFAA-R, NRF54L15-QFAA-R:QFN40P600X600X90-49N, symbol NRF54L15-QFAA-R:NRF54L15-QFAA-R
- added Y2: 32 MHz, symbol Device:Crystal
Connections:
- net GND: now also C22.2, C23.2, C24.2, C25.2, C26.2, C27.2, C28.2, C29.2, C30.2, C31.2, C33.2, C34.2, C36.1, U6.44 (VSS), U6.49 (VSS)
- net MISO_OUT: now also U6.13 (P2.02)
- net MOSI_OUT: now also U6.15 (P2.04)
- net SCLK_OUT: now also U6.12 (P2.01)
- net at U1.23 (VREF): now also C36.2
- new net: C32.1, L2.2, L3.1
- new net: C33.1, L3.2, L4.1
- new net: C34.1, L4.2
- new net: C22.1, R7.1
- new net: U6.34 (XC1), Y2.2
- new net: U6.35 (XC2), Y2.1
- new net: J4.A1 (GND), J4.A12 (GND), J4.B1 (GND), J4.B12 (GND)
- new net: J4.A4 (VBUS), J4.A9 (VBUS), J4.B4 (VBUS), J4.B9 (VBUS)
- new net ANT: L2.1, U6.31 (ANT)
- new net DCC: L1.1, U6.46 (DCC)
- new net DEBUG_D+: J4.A6 (D+), J4.B6 (D+)
- new net DEBUG_D-: J4.A7 (D-), J4.B7 (D-)
- new net DECA: C29.1, C30.1, C31.1, FB1.1, U6.33 (DECRF), U6.43 (DECA)
- new net DECD: C28.1, FB1.2, L1.2, U6.45 (DECD)
- new net NRESET: R7.2, U6.30 (~{RESET})
- new net VDD: C23.1, C24.1, C25.1, C26.1, C27.1, U6.10 (VDD), U6.22 (VDD), U6.36 (VDD), U6.47 (VDD), U6.48 (VDD)
- new net VSS_PA: C32.2, U6.32 (VSS_PA)
Other:
- note added: "FUEL GAUGE"
- note removed: "BMS"
- moved on the sheet: C1, C10, C12, C13, C14, C15, C16, C19, C2, C20, C3, C4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
