File: MCU_V2/MCU_V2.kicad_pcb (KiCad board)
At the start: 2 copper layers, 63 x 28 mm, 11 parts, among them J2 Conn_01x09_Pin, J3 Conn_01x02_Socket, U1 XIAO-nRF54l15-SMD, U5 MAX17048G_T10

Commit message: six seven
Parts:
- added G***: LOGO, LOGO, B.Cu at (207.5, 97.8)
Other:
- board text added: "Rev 5.0"
- board text added: "designed by Daksh V."
